File: pcb/ergoslab.sch (KiCad schematic (older format))
At the start: 78 parts, among them J1 L_B_LED, J2 R_B_LED, J3 SLAVE_LED, P1 OLED, P2 ICSP, SW0:0 SW_Push, SW0:1 SW_Push, SW0:2 SW_Push, SW0:3 SW_Push, SW0:4 SW_Push, SW1:0 SW_Push, SW1:1 SW_Push, SW1:2 SW_Push, SW1:3 SW_Push, SW1:4 SW_Push, SW2:0 SW_Push, SW2:1 SW_Push, SW2:2 SW_Push, SW2:3 SW_Push, SW2:4 SW_Push, SW3:0 SW_Push, SW3:1 SW_Push, SW3:2 SW_Push, SW3:3 SW_Push, SW3:4 SW_Push, SW3:5 SW_Push, SW4:1 SW_Push, SW4:2 SW_Push, SW4:3 SW_Push, SW4:4 SW_Push, SW4:5 SW_Push

Commit message: refactor: house clean unused symbols and footprints, merge all symbols into one library, rename kicad project from testy to ergoslab
Parts:
- JP1, JP10, JP11, JP12, JP2, JP3, JP4, JP5, JP6, JP7, JP8, JP9: symbol jp2:JP2 -> this_keeb:JP2
- LED_L1, LED_R1: symbol sk6812mini:SK6812mini -> this_keeb:SK6812mini
- P1: symbol conn_01x04:CONN_01X04 -> this_keeb:CONN_01X04
- P2: symbol conn_01x06:CONN_01X06 -> this_keeb:CONN_01X06
- PM1: symbol promicro:ProMicro -> this_keeb:ProMicro
- R1, R2: symbol resistor:R -> this_keeb:R
- TRRS1: symbol mj-4pp-9:MJ-4PP-9 -> this_keeb:MJ-4PP-9
Changed lines of the file:
@@
 EESchema Schematic File Version 4
-LIBS:testy-cache
+LIBS:ergoslab-cache
 EELAYER 30 0
 EELAYER END
@@
 Row2
 $Comp
-L promicro:ProMicro PM1
+L this_keeb:ProMicro PM1
 U 1 1 5DB7A2E7
 P 1750 2250
@@
 Row3
 $Comp
-L mj-4pp-9:MJ-4PP-9 TRRS1
+L this_keeb:MJ-4PP-9 TRRS1
 U 1 1 5DB680F2
 P 2150 7200
@@
 SCL
 $Comp
-L conn_01x04:CONN_01X04 P1
+L this_keeb:CONN_01X04 P1
 U 1 1 5DCD19CA
 P 4050 5700
@@
 $EndComp
 $Comp
-L jp2:JP2 JP1
+L this_keeb:JP2 JP1
 U 1 1 5DCEEF2E
 P 4950 5400
@@
 $EndComp
 $Comp
-L jp2:JP2 JP2
+L this_keeb:JP2 JP2
 U 1 1 5DCF00CE
 P 4950 5600
@@
 $EndComp
 $Comp
-L jp2:JP2 JP4
+L this_keeb:JP2 JP4
 U 1 1 5DCF0797
 P 4950 6000
@@
 $EndComp
 $Comp
-L jp2:JP2 JP3
+L this_keeb:JP2 JP3
 U 1 1 5DCF0E97
 P 4950 5800
@@
 SDA
 $Comp
-L jp2:JP2 JP8
+L this_keeb:JP2 JP8
 U 1 1 5DD6CDF9
 P 4950 7000
@@
 $EndComp
 $Comp
-L jp2:JP2 JP7
+L this_keeb:JP2 JP7
 U 1 1 5DD6CE03
 P 4950 6800
@@
 $EndComp
 $Comp
-L jp2:JP2 JP5
+L this_keeb:JP2 JP5
 U 1 1 5DD6CE0D
 P 4950 6400
@@
 $EndComp
 $Comp
-L jp2:JP2 JP6
+L this_keeb:JP2 JP6
 U 1 1 5DD6CE17
 P 4950 6600
@@
 Left hand side
 $Comp
-L conn_01x06:CONN_01X06 P2
+L this_keeb:CONN_01X06 P2
 U 1 1 5DDC8800
 P 6550 5750
@@
 	3650 4650 5650 4650
 $Comp
-L sk6812mini:SK6812mini LED_L1
+L this_keeb:SK6812mini LED_L1
 U 1 1 5DE1DE41
 P 2050 5100
@@
 LED
 $Comp
-L resistor:R R1
+L this_keeb:R R1
 U 1 1 5DE28F05
 P 8350 5400
@@
 $EndComp
 $Comp
-L resistor:R R2
+L this_keeb:R R2
 U 1 1 5DE296C1
 P 8750 5400
@@
 SDA
 $Comp
-L sk6812mini:SK6812mini LED_R1
+L this_keeb:SK6812mini LED_R1
 U 1 1 5DE5B1E3
 P 2050 6350
@@
 $EndComp
 $Comp
-L jp2:JP2 JP9
+L this_keeb:JP2 JP9
 U 1 1 5DE66916
 P 2000 5650
@@
 SLAVE_LED
 $Comp
-L jp2:JP2 JP12
+L this_keeb:JP2 JP12
 U 1 1 5DF1D947
 P 2000 5900
@@
 For info about PWR_FLAG, see https://forum.kicad.info/t/errtype-3-pin-connected-to-some-others-pins-but-no-pin-to-drive-it/10946
 $Comp
-L jp2:JP2 JP11
+L this_keeb:JP2 JP11
 U 1 1 5DEDAECF
 P 2950 5900
@@
 Connection ~ 3150 5750
 $Comp
-L jp2:JP2 JP10
+L this_keeb:JP2 JP10
 U 1 1 5DEF3C70
 P 2950 5650
